File: master_side.kicad_sch (KiCad schematic)
At the start: 49 parts, among them J1 AudioJack4, J2 Conn_01x02, J3 Conn_02x18_Odd_Even, J4 Conn_02x18_Odd_Even, J5 USB_C_Receptacle_USB2.0_14P, Q1 Q_NMOS, U1 W25Q128JVS, U2 NCP1117-3.3_SOT223, U3 RP2040, U4 BH1750FVI-TR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

Commit message: Add TRRS connector, rotary encoder, ambient light sensor
Parts:
- removed R10: R_Photo, symbol Device:R_Photo
- removed U4: BH1750FVI-TR, BH1750FVI-TR:XDCR_BH1750FVI-TR, symbol BH1750FVI-TR:BH1750FVI-TR
- added C18: 100n, symbol library:C
- added R10, R11: 3.3k, symbol library:R
- added R12, R13: 33, symbol library:R
- added SW1: RotaryEncoder, symbol Device:RotaryEncoder
- added SW2: SW_Push, symbol Switch:SW_Push
- added TP5: TestPoint, symbol Connector:TestPoint
- added U4: OPT3001DNPR, Package_TO_SOT_SMD:SOT-223-3_TabPin2, symbol OPT3001DNPR:OPT3001DNPR
Connections:
- net +3V3: now also C18.1, R10.1, R11.1, U4.1 (VDD)
- net GND: now also C18.2, SW1.B, SW2.2, U4.2 (ADDR), U4.3 (GND)
- net GPIO2: now also R12.1; no longer R9.1
- net GPIO3: now also R13.1; no longer R8.1
- net GPIO4: now also R9.1
- net GPIO5: now also R8.1
- net GPIO6: now also U3.8 (GPIO6), SW1.A
- net GPIO7: now also U3.9 (GPIO7), SW1.C
- net GPIO8: now also U3.11 (GPIO8), SW2.1
- new net: R10.2, R12.2, U4.6 (SDA)
- new net: R11.2, R13.2, U4.4 (SCL)
- new net: TP5.1, U4.5 (INT)
Other:
- note added: "ambient light sensor for backlight dimming"
- note added: "do not connect"
- note added: "interrupt pin (unused, since polling from RP2040 over I2C)"
- note added: "make sure cap is close to IC"
- note added: "status LEDs"
- note added: "volume knob"
- moved on the sheet: D1, D2, R8, R9
