File: pcb/slave_side.kicad_sch (KiCad schematic)
At the start: 71 parts, among them IC2 PCA9956BTWY, J4 4P4C, SW20 SW_Push_45deg, SW21 SW_Push_45deg, SW22 SW_Push_45deg, SW23 SW_Push_45deg, SW24 SW_Push_45deg, SW25 SW_Push_45deg, SW26 SW_Push_45deg, SW27 SW_Push_45deg, SW28 SW_Push_45deg, SW29 SW_Push_45deg, SW30 SW_Push_45deg, SW31 SW_Push_45deg, SW32 SW_Push_45deg, SW33 SW_Push_45deg, SW34 SW_Push_45deg, SW35 SW_Push_45deg, SW36 SW_Push_45deg, SW37 SW_Push_45deg, U5 MCP23017T-E/ML, U6 NCP1117LPST33T3G, U7 OPT3001DNPR

Commit message: fix: PCA9956 OE pin and RESET pin and improve LED power delivery
Parts:
- added C23: 10u, symbol Device:C
- F3: footprint (none) -> Fuse:Fuse_1206_3216Metric
- renumbered C18 to C19, C19 to C20, C20 to C21, C21 to C22, J4 to J3, R15 to R16, R16 to R17, R17 to R18, SW20 to SW21, SW21 to SW22, SW22 to SW23, SW23 to SW24, SW24 to SW25, SW25 to SW26, SW26 to SW27, SW27 to SW28, SW28 to SW29, SW29 to SW30, SW30 to SW31, SW31 to SW32, SW32 to SW33, SW33 to SW34, SW34 to SW35, SW35 to SW36, SW36 to SW37, SW37 to SW38
Connections:
- net +3V3_R: no longer R16.1
- net +5V_R: now also C23.1
Other:
- note removed: "EXP is the heatsink under the IC, make many thermal vias under the chip"

Commit message: fix: Diode & switch numbering for kbplacer
Parts:
- added C23, C24: 100n, Capacitor_SMD:C_0805_2012Metric, symbol Device:C
- added R17: 10k, Resistor_SMD:R_0402_1005Metric, symbol library:R
- C26: renamed from C23; footprint (none) -> Capacitor_SMD:C_0805_2012Metric
- renumbered C19 to C25, D38 to D21, D39 to D22, D40 to D23, D41 to D24, D42 to D25, D43 to D26, D44 to D27, D45 to D28, D46 to D29, D47 to D30, D48 to D31, D49 to D32, D50 to D33, D51 to D34, D52 to D35, D53 to D36, D54 to D37, D55 to D38, D61 to D39, D63 to D40, D65 to D41, D56 to LD19, D57 to LD20, D58 to LD21, D59 to LD22, D60 to LD23, D62 to LD24, D64 to LD25, D66 to LD26, D67 to LD27, D68 to LD28, D69 to LD29, D70 to LD30, D71 to LD31, D72 to LD32, D73 to LD33, D74 to LD34, D75 to LD35, D76 to LD36, R16 to R18, R17 to R19, R18 to R20, SW21 to SW22, SW22 to SW23, SW23 to SW24, SW24 to SW25, SW25 to SW26, SW26 to SW27, SW27 to SW28, SW28 to SW29, SW29 to SW30, SW30 to SW31, SW31 to SW32, SW32 to SW33, SW33 to SW34, SW34 to SW35, SW35 to SW36, SW36 to SW37, SW37 to SW38, SW38 to SW39, U6 to U5, U5 to U6
Connections:
- net +3V3_R: now also C23.2, C24.2, R17.1
- net ROW1R: now also D21.1 (K), D22.1 (K), D23.1 (K), D24.1 (K), D25.1 (K), D26.1 (K); no longer D21.2 (A), D22.2 (A), D23.2 (A), D24.2 (A), D25.2 (A), D26.2 (A)
- net ROW2R: now also D27.1 (K), D28.1 (K), D29.1 (K), D30.1 (K), D31.1 (K), D32.1 (K); no longer D27.2 (A), D28.2 (A), D29.2 (A), D30.2 (A), D31.2 (A), D32.2 (A)
- net ROW3R: now also D33.1 (K), D34.1 (K), D35.1 (K), D36.1 (K), D37.1 (K), D38.1 (K); no longer D33.2 (A), D34.2 (A), D35.2 (A), D36.2 (A), D37.2 (A), D38.2 (A)
- net at SW37.2: now also D36.2 (A); no longer D36.1 (K)
- net at SW24.2: now also D23.2 (A); no longer D23.1 (K)
- net at SW30.2: now also D29.2 (A); no longer D29.1 (K)
- net at SW34.2: now also D33.2 (A); no longer D33.1 (K)
- net at SW27.2: now also D26.2 (A); no longer D26.1 (K)
- net at SW35.2: now also D34.2 (A); no longer D34.1 (K)
- net at SW22.2: now also D21.2 (A); no longer D21.1 (K)
- net at SW23.2: now also D22.2 (A); no longer D22.1 (K)
- net at SW38.2: now also D37.2 (A); no longer D37.1 (K)
- net at SW32.2: now also D31.2 (A); no longer D31.1 (K)
- net at SW25.2: now also D24.2 (A); no longer D24.1 (K)
- net at SW36.2: now also D35.2 (A); no longer D35.1 (K)
- net at SW29.2: now also D28.2 (A); no longer D28.1 (K)
- net at SW31.2: now also D30.2 (A); no longer D30.1 (K)
- net at SW28.2: now also D27.2 (A); no longer D27.1 (K)
- net at U6.14 (*RESET): now also R17.2
- net at SW26.2: now also D25.2 (A); no longer D25.1 (K)
- net at SW39.2: now also D38.2 (A); no longer D38.1 (K)
- net at SW33.2: now also D32.2 (A); no longer D32.1 (K)
Other:
- note added: "4p4c port & 5v to 3.3v stepdown"
- note added: "backlight LED driver"
- moved on the sheet: C20, C21, C22, C25, C26, D21, D22, D23, D24, D25, D26, D27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

Commit message: fix: Proper USB-C receptacle symbol
Parts:
- removed C20: 20u, Capacitor_SMD:C_0805_2012Metric, symbol Device:C
- renumbered C21 to C20, C22 to C21, C23 to C22, C24 to C23, C25 to C24, C26 to C25, SW22 to SW19, SW23 to SW20, SW24 to SW21, SW25 to SW22, SW26 to SW23, SW27 to SW24, SW28 to SW25, SW29 to SW26, SW30 to SW27, SW31 to SW28, SW32 to SW29, SW33 to SW30, SW34 to SW31, SW35 to SW32, SW36 to SW33, SW37 to SW34, SW38 to SW35, SW39 to SW36

Commit message: fix: Fix thumb cluster key splay & Correctly align keys to outline in PCB layout
Parts:
- U7: DESCRIPTION Digital ambient light sensor (ALS) with high-precision huma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 -> (none)
Connections:
- net COL1R renamed COL6
- net COL6: now also U6.25 (GPB0); no longer U6.20 (GPA3)
- net COL2R renamed COL7
- net COL7: now also U6.24 (GPA7); no longer U6.21 (GPA4)
- net COL3R renamed COL8
- net COL8: now also U6.23 (GPA6); no longer U6.22 (GPA5)
- net COL4R renamed COL9
- net COL9: now also U6.22 (GPA5); no longer U6.23 (GPA6)
- net COL5R renamed COL10
- net COL10: now also U6.21 (GPA4); no longer U6.24 (GPA7)
- net COL6R renamed COL11
- net COL11: now also U6.20 (GPA3); no longer U6.25 (GPB0)
- net ROW1R renamed ROW0
- net ROW0: now also U6.19 (GPA2); no longer U6.17 (GPA0)
- net ROW2R renamed ROW1
- net ROW3R renamed ROW2
- net ROW2: now also U6.17 (GPA0); no longer U6.19 (GPA2)

Commit message: feat: Add NC flags to both side schematics
Connections:
- no-connect marks 0 -> 14
Changed lines of the file:
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@@
 		(color 0 0 0 0)
+	)
+	(no_connect
+		(at 274.32 83.82)
+	)
+	(no_connect
+		(at 228.6 81.28)
+	)
+	(no_connect
+		(at 116.84 193.04)
+	)
+	(no_connect
+		(at 274.32 86.36)
+	)
+	(no_connect
+		(at 116.84 190.5)
+	)
+	(no_connect
+		(at 116.84 187.96)
+	)
+	(no_connect
+		(at 228.6 104.14)
+	)
+	(no_connect
+		(at 274.32 116.84)
+	)
+	(no_connect
+		(at 228.6 86.36)
+	)
+	(no_connect
+		(at 274.32 114.3)
+	)
+	(no_connect
+		(at 228.6 83.82)
+	)
+	(no_connect
+		(at 228.6 88.9)
+	)
+	(no_connect
+		(at 228.6 96.52)
+	)
+	(no_connect
+		(at 281.94 191.77)
 	)
 	(wire
