File: pcb/slave_side.kicad_sch (KiCad schematic)
At the start: 74 parts, among them IC2 PCA9956BTWY, J3 4P4C, SW19 SW_Push_45deg, SW20 SW_Push_45deg, SW21 SW_Push_45deg, SW22 SW_Push_45deg, SW23 SW_Push_45deg, SW24 SW_Push_45deg, SW25 SW_Push_45deg, SW26 SW_Push_45deg, SW27 SW_Push_45deg, SW28 SW_Push_45deg, SW29 SW_Push_45deg, SW30 SW_Push_45deg, SW31 SW_Push_45deg, SW32 SW_Push_45deg, SW33 SW_Push_45deg, SW34 SW_Push_45deg, SW35 SW_Push_45deg, SW36 SW_Push_45deg, U5 NCP1117LPST33T3G, U6 MCP23017T-E/ML, U7 OPT3001DNPR

Commit message: feat: Add screw mount holes, add more JLC part numbers, fix DRC violations, remove all components at least 1mm from the edge of the board, add Cherry switch 3D model to ai03 footprint
Connections:
- net +3V3_R: now also IC2.3 (AD1)
- net at IC2.2 (AD0), IC2.4 (AD2): no longer IC2.3 (AD1)
Changed lines of the file:
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@@
 	)
 	(junction
-		(at 68.58 177.8)
-		(diameter 0)
-		(color 0 0 0 0)
-	)
-	(junction
 		(at 359.41 120.65)
 		(diameter 0)
@@
 	(wire
 		(pts
-			(xy 68.58 175.26) (xy 71.12 175.26)
+			(xy 63.5 175.26) (xy 71.12 175.26)
 		)
 		(stroke
@@
 	(wire
 		(pts
-			(xy 68.58 180.34) (xy 68.58 177.8)
+			(xy 63.5 175.26) (xy 63.5 180.34)
 		)
 		(stroke
@@
 	(wire
 		(pts
-			(xy 64.77 177.8) (xy 68.58 177.8)
-		)
-		(stroke
-			(width 0)
-			(type default)
-		)
-	)
-	(wire
-		(pts
 			(xy 59.69 210.82) (xy 66.04 210.82)
 		)
@@
 	(wire
 		(pts
-			(xy 68.58 177.8) (xy 71.12 177.8)
-		)
-		(stroke
-			(width 0)
-			(type default)
-		)
-	)
-	(wire
-		(pts
 			(xy 347.98 106.68) (xy 359.41 106.68)
 		)
@@
 	(wire
 		(pts
-			(xy 68.58 177.8) (xy 68.58 175.26)
-		)
-		(stroke
-			(width 0)
-			(type default)
-		)
-	)
-	(wire
-		(pts
 			(xy 308.61 82.55) (xy 308.61 96.52)
 		)
@@
 	(wire
 		(pts
-			(xy 71.12 180.34) (xy 68.58 180.34)
+			(xy 71.12 180.34) (xy 63.5 180.34)
 		)
 		(stroke
@@
 		(length 2.54)
 		(shape round)
-		(at 64.77 177.8 90)
+		(at 63.5 177.8 90)
 		(effects
 			(font
@@
 		)
 		(property "Net Class" "R_GND"
-			(at 60.96 177.8 0)
+			(at 59.69 177.8 0)
 			(show_name no)
 			(do_not_autoplace no)
@@
 		)
 		(property "Component Class" ""
-			(at 160.02 -115.57 90)
+			(at 158.75 -115.57 90)
 			(show_name no)
 			(do_not_autoplace no)
@@
 					(unit 1)
 				)
+			)
+		)
+	)
+	(symbol
+		(lib_id "power:+3V3")
+		(at 71.12 177.8 90)
+		(unit 1)
+		(body_style 1)
+		(exclude_from_sim no)
+		(in_bom yes)
+		(on_board yes)
+		(in_pos_files yes)
+		(dnp no)
+		(property "Reference" "#PWR060"
+			(at 74.93 177.8 0)
+			(hide yes)
+			(show_name no)
+			(do_not_autoplace no)
+			(effects
+				(font
+					(size 1.27 1.27)
+				)
+			)
+		)
+		(property "Value" "+3V3_R"
+			(at 63.5 179.07 90)
+			(show_name no)
+			(do_not_autoplace no)
+			(effects
+				(font
+					(size 1.27 1.27)
+				)
+				(justify right)
+			)
+		)
+		(property "Footprint" ""
+			(at 71.12 177.8 0)
+			(hide yes)
+			(show_name no)
+			(do_not_autoplace no)
+			(effects
+				(font
+					(size 1.27 1.27)
+				)
+			)
+		)
+		(property "Datasheet" ""
+			(at 71.12 177.8 0)
+			(hide yes)
+			(show_name no)
+			(do_not_autoplace no)
+			(effects
+				(font
+					(size 1.27 1.27)
+				)
+			)
+		)
+		(property "Description" "Power symbol creates a global label with name \"+3V3\""
+			(at 71.12 177.8 0)
+			(hide yes)
+			(show_name no)
+			(do_not_autoplace no)
+			(effects
+				(font
+					(size 1.27 1.27)
+				)
+			)
+		)
+		(pin "1"
+		)
+		(instances
+			(project "mSCKee"
+				(path "/2ec7cb33-7d00-426e-b710-cc42b1f2f810/84141690-5233-4517-90f0-209001a553bd"
+					(reference "#PWR060")
+					(unit 1)
+				)

Commit message: fix: Size all footprints on the back side 0805 for hand soldering
Parts:
- R18: value 2k -> 3k
Other:
- note added: "I2C: 0010101"
- note removed: "I2C: 0000001"
Changed lines of the file:
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@@
 		)
 	)
+	(text "I2C: 0010101"
+		(exclude_from_sim no)
+		(at 92.71 157.48 0)
+		(effects
+			(font
+				(size 1.27 1.27)
+			)
+		)
+	)
 	(text "same I2C adress as the LED driver on master side, \nbut using different I2C bus, so no conflict"
 		(exclude_from_sim no)
@@
 		)
 	)
-	(text "I2C: 0000001"
-		(exclude_from_sim no)
-		(at 92.71 157.48 0)
-		(effects
-			(font
-				(size 1.27 1.27)
-			)
-		)
-	)
 	(text "NC = not connected"
 		(exclude_from_sim no)
@@
 			)
 		)
-		(property "Value" "2k"
+		(property "Value" "3k"
 			(at 69.85 170.18 90)
 			(show_name no)
