File: pcb/master_side.kicad_sch (KiCad schematic)
At the start: 109 parts, among them IC1 PCA9956BTWY, J2 4P4C, J4 USB_C_Receptacle_USB2.0_16P, SW1 SW_Push_45deg, SW10 SW_Push_45deg, SW11 SW_Push_45deg, SW12 SW_Push_45deg, SW13 SW_Push_45deg, SW14 SW_Push_45deg, SW15 SW_Push_45deg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

Commit message: feat: Improve layout & route crystal and flash
Parts:
- C1, C2, C3, C4, C5, C6, C7: footprint Capacitor_SMD:C_0805_2012Metric -> Capacitor_SMD:C_0402_1005Metric
- C10, C11: footprint Capacitor_SMD:C_01005_0402Metric -> Capacitor_SMD:C_0402_1005Metric
- R15, R16: footprint Resistor_SMD:R_0402_1005Metric -> Resistor_SMD:R_0201_0603Metric
Changed lines of the file:
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@@
 			)
 		)
-		(property "Footprint" "Capacitor_SMD:C_0805_2012Metric"
+		(property "Footprint" "Capacitor_SMD:C_0402_1005Metric"
 			(at 233.3752 45.72 0)
 			(hide yes)
@@
 			)
 		)
-		(property "Footprint" "Capacitor_SMD:C_0805_2012Metric"
+		(property "Footprint" "Capacitor_SMD:C_0402_1005Metric"
 			(at 244.8052 45.72 0)
 			(hide yes)
@@
 			)
 		)
-		(property "Footprint" "Capacitor_SMD:C_0805_2012Metric"
+		(property "Footprint" "Capacitor_SMD:C_0402_1005Metric"
 			(at 256.2352 45.72 0)
 			(hide yes)
@@
 			)
 		)
-		(property "Footprint" "Capacitor_SMD:C_0805_2012Metric"
+		(property "Footprint" "Capacitor_SMD:C_0402_1005Metric"
 			(at 267.6652 45.72 0)
 			(hide yes)
@@
 			)
 		)
-		(property "Footprint" "Capacitor_SMD:C_0805_2012Metric"
+		(property "Footprint" "Capacitor_SMD:C_0402_1005Metric"
 			(at 279.0952 45.72 0)
 			(hide yes)
@@
 			)
 		)
-		(property "Footprint" "Capacitor_SMD:C_0805_2012Metric"
+		(property "Footprint" "Capacitor_SMD:C_0402_1005Metric"
 			(at 290.5252 45.72 0)
 			(hide yes)
@@
 			)
 		)
-		(property "Footprint" "Capacitor_SMD:C_0805_2012Metric"
+		(property "Footprint" "Capacitor_SMD:C_0402_1005Metric"
 			(at 301.9552 45.72 0)
 			(hide yes)
@@
 			)
 		)
-		(property "Footprint" "Capacitor_SMD:C_01005_0402Metric"
+		(property "Footprint" "Capacitor_SMD:C_0402_1005Metric"
 			(at 178.7652 77.47 0)
 			(hide yes)
@@
 			)
 		)
-		(property "Footprint" "Capacitor_SMD:C_01005_0402Metric"
+		(property "Footprint" "Capacitor_SMD:C_0402_1005Metric"
 			(at 215.5952 64.77 0)
 			(hide yes)
@@
 			)
 		)
-		(property "Footprint" "Resistor_SMD:R_0402_1005Metric"
+		(property "Footprint" "Resistor_SMD:R_0201_0603Metric"
 			(at 180.34 248.158 90)
 			(hide yes)
@@
 			)
 		)
-		(property "Footprint" "Resistor_SMD:R_0402_1005Metric"
+		(property "Footprint" "Resistor_SMD:R_0201_0603Metric"
 			(at 180.34 234.188 90)
 			(hide yes)

Commit message: feat: Add NC flags to both side schematics
Connections:
- no-connect marks 0 -> 18
Changed lines of the file:
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@@
 		(color 0 0 0 0)
+	)
+	(no_connect
+		(at 104.14 229.87)
+	)
+	(no_connect
+		(at 238.76 162.56)
+	)
+	(no_connect
+		(at 238.76 157.48)
+	)
+	(no_connect
+		(at 238.76 165.1)
+	)
+	(no_connect
+		(at 104.14 224.79)
+	)
+	(no_connect
+		(at 238.76 177.8)
+	)
+	(no_connect
+		(at 238.76 180.34)
+	)
+	(no_connect
+		(at 238.76 167.64)
+	)
+	(no_connect
+		(at 238.76 160.02)
+	)
+	(no_connect
+		(at 104.14 222.25)
+	)
+	(no_connect
+		(at 238.76 172.72)
+	)
+	(no_connect
+		(at 238.76 175.26)
+	)
+	(no_connect
+		(at 351.79 213.36)
+	)
+	(no_connect
+		(at 104.14 234.95)
+	)
+	(no_connect
+		(at 238.76 152.4)
+	)
+	(no_connect
+		(at 104.14 232.41)
+	)
+	(no_connect
+		(at 104.14 227.33)
+	)
+	(no_connect
+		(at 238.76 154.94)
 	)
 	(wire

Commit message: chore: Restructure Journal (import from fallout) for outpost
Parts:
- F1: value Polyfuse_Small -> 500mA
Changed lines of the file:
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@@
 		(fields_autoplaced yes)
 		(property "Reference" "F1"
-			(at 284.48 116.8399 0)
+			(at 284.48 116.84 0)
 			(show_name no)
 			(do_not_autoplace no)
@@
 			)
 		)
-		(property "Value" "Polyfuse_Small"
-			(at 284.48 119.3799 0)
+		(property "Value" "500mA"
+			(at 284.48 119.38 0)
 			(show_name no)
 			(do_not_autoplace no)
